File: hardware/inside_board/heimdall_insideboard.sch (KiCad schematic (older format))
At the start: 58 parts, among them J1 Barrel_Jack_Switch, J2 Screw_Terminal_01x04, J3 Conn_01x09, J4 Screw_Terminal_01x04, J5 Conn_01x09, J6 Screw_Terminal_01x04, J7 Screw_Terminal_01x06, J8 Screw_Terminal_01x09, J9 Screw_Terminal_01x02, K1 Relay_HJR-3FF-S-Z-5VDC, K2 Relay_HJR-3FF-S-Z-5VDC, K3 Relay_HJR-3FF-S-Z-5VDC, Q1 2N3904, Q2 2N3904, Q3 2N3904, Q4 2N3904, Q5 2N3904, Q6 2N3904, U1 LM1117-3.3, U2 L7805, U3 ESP32_Dev_Board_30Pin

Commit message: Update heimdall_insideboard.sch with version from Steven Hildebrand
Steven Hildebrand has improved the layout of the inside board schematic
to avoid overlapping text and symbols.
Parts:
- removed R10, R11, R12, R13, R14, R2, R3, R4, R5, R7, R8, R9: 220, Resistor_THT:R_Axial_DIN0207_L6.3mm_D2.5mm_P10.16mm_Horizontal, symbol Device:R_Small_US
- removed U3: ESP32_Dev_Board_30Pin, Javawizard_Common_Footprints:JW_ESP32_DevKit_30Pin, symbol heimdall_insideboard-rescue:ESP32_Dev_Board_30Pin-Javawizard_Common_Schematic_S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
- added R10, R11, R12, R13, R14, R2, R3, R4, R5, R7, R8, R9: 220, symbol Device:R_US
- added U3: ESP32_Dev_Board_30Pin, symbol heimdall_insideboard-rescue:ESP32_Dev_Board_30Pin-Javawizard_Common_Schematic_S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
- C1, C2, C3: value 22uF -> 22µF
- K1, K2, K3: symbol heimdall_insideboard-rescue:Relay_HJR-3FF-S-Z-5VDC-Javawizard_Common_Schematic_Symbols -> heimdall_insideboard-rescue:Relay_HJR-3FF-S-Z-5VDC-Javawizard_Common_Schematic_Symbols-heimdall_insideboard-rescue
- R16, R17, R25: value 1k5 -> 1.5k
- R18, R20, R22, R23, R24: value 2k2 -> 2.2k
Connections:
- net labels added: +3.3V
- net labels removed: +3V3
- wire segments 280 -> 274
Other:
- note added: "+3.3v"
- note added: "+5v"
- note added: "GND"
- note added: "U3-10\nMISO"
- note added: "U3-25\nLED"
- note added: "U3-26\nBeeper"
- note added: "U3-29\nLED"
- note added: "U3-30\nBeeper"
- note added: "U3-6\nCS"
- note added: "U3-7\nCS"
- note added: "U3-8\nSCK"
- note added: "U3-9\nMOSI"
