File: hardware/outside_boards/antenna/antenna.kicad_pcb (KiCad board)
At the start: 2 copper layers, 70 x 100 mm, 10 parts, among them J1 Jumper, J2 Conn_01x03_Pin

Commit message: Finished layout, probably?
Parts:
- added REF**: MountingHole_4.3mm_M4, MountingHole:MountingHole_4.3mm_M4, F.Cu at (173.0, 80.0)
- added REF**: MountingHole_4.3mm_M4, MountingHole:MountingHole_4.3mm_M4, F.Cu at (113.0, 80.0)
- moved REF** 15.0 mm to (173.0, 110.0)
- moved REF** 15.0 mm to (113.0, 110.0)
Other:
- board text added: "Heimdall Reader (CLRC663) Make Salt Lake August 2025 https://github.com/makesaltlake/heimdall Antenna V0"
